File: PCI_104_PCIE_Adapterboard.kicad_pcb (KiCad board)
At the start: 2 copper layers, 52 parts, among them J1 ASP-129637-03, J10 1-2199119-5, J2 10061913-102PLF, J3 Conn_01x02_Pin, J4 Conn_01x02_Pin, J5 Conn_01x02_Pin, J6 10061913-102PLF, J7 1-2199119-5, J8 1-2199119-5, J9 1-2199119-5, U1 ZL40264LDG1, U2 TPS54KB21RZRR

Commit message: pcie traces routed
Parts:
- added C21: 10uF, Capacitor_SMD:C_0805_2012Metric_Pad1.18x1.45mm_HandSolder, F.Cu at (287.0, 33.5)
- added C22: 10uF, Capacitor_SMD:C_0805_2012Metric_Pad1.18x1.45mm_HandSolder, F.Cu at (287.0, 36.5)
- added C23: 10uF, Capacitor_SMD:C_0805_2012Metric_Pad1.18x1.45mm_HandSolder, F.Cu at (287.0, 39.5)
- added C24: 10uF, Capacitor_SMD:C_0805_2012Metric_Pad1.18x1.45mm_HandSolder, F.Cu at (287.0, 42.5)
- added C25: 10uF, Capacitor_SMD:C_0805_2012Metric_Pad1.18x1.45mm_HandSolder, F.Cu at (287.0, 45.5)
- added C26: 10uF, Capacitor_SMD:C_0805_2012Metric_Pad1.18x1.45mm_HandSolder, F.Cu at (287.0, 48.5)
- added C27: 10uF, Capacitor_SMD:C_0805_2012Metric_Pad1.18x1.45mm_HandSolder, F.Cu at (287.0, 51.6)
- added C28: 10uF, Capacitor_SMD:C_0805_2012Metric_Pad1.18x1.45mm_HandSolder, F.Cu at (287.0, 54.6)
- added C29: 10uF, Capacitor_SMD:C_1206_3216Metric, F.Cu at (294.2, 33.7)
- added C30: 10uF, Capacitor_SMD:C_0805_2012Metric_Pad1.18x1.45mm_HandSolder, F.Cu at (299.4, 33.5)
- added C31: 10uF, Capacitor_SMD:C_1206_3216Metric, F.Cu at (294.2, 37.0)
- added C32: 10uF, Capacitor_SMD:C_1206_3216Metric, F.Cu at (294.2, 40.4)
- added H1: MountingHole_Pad, MountingHole:MountingHole_3.2mm_M3_Pad_TopBottom, F.Cu at (35.0, 35.7)
- added H2: MountingHole_Pad, MountingHole:MountingHole_3.2mm_M3_Pad_TopBottom, F.Cu at (120.7, 33.2)
- added H3: MountingHole_Pad, MountingHole:MountingHole_3.2mm_M3_Pad_TopBottom, F.Cu at (35.0, 109.4)
- added H4: MountingHole_Pad, MountingHole:MountingHole_3.2mm_M3_Pad_TopBottom, F.Cu at (120.7, 113.2)
- added J11: Conn_01x02_Pin, Connector_PinHeader_2.54mm:PinHeader_1x02_P2.54mm_Vertical, F.Cu at (261.8, 29.2)
- added L1: 150nH, footprints:INDPM5350X200N, F.Cu at (263.8, 148.9)
- C12, C13, C15, C16, C2, C3, C4, C5, C7, C8: footprint Capacitor_SMD:C_0201_0603Metric_Pad0.64x0.40mm_HandSolder -> Capacitor_SMD:C_0603_1608Metric
- moved J3 213.2 mm to (282.3, 106.4)
- moved U1 213.2 mm to (289.6, 75.4)
- moved C2 164.3 mm to (340.0, 113.7)
- moved C3 164.3 mm to (340.0, 115.4)
- moved C4 164.3 mm to (340.0, 117.2)
- moved C5 164.3 mm to (340.0, 118.9)
- moved R16 160.2 mm to (311.1, 165.8)
- moved R17 160.2 mm to (311.1, 168.3)
- moved C12 153.5 mm to (328.7, 145.8)
- moved C13 153.5 mm to (328.7, 147.5)
- moved C7 153.5 mm to (325.9, 152.8)
- moved C8 153.5 mm to (325.9, 154.5)
- moved C10 153.5 mm to (311.9, 155.4)
- moved C11 153.5 mm to (311.9, 158.5)
- moved C17 153.5 mm to (316.7, 149.4)
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Connections:
- net /DIR renamed /PCIe 104/DIR
- net /PE_RST# renamed PE_RST#
- net /PEx16_0R(10)_N renamed PEx16_0R(10)_N
- net /PEx16_0R(10)_P renamed PEx16_0R(10)_P
- net /PEx16_0R(11)_N renamed PEx16_0R(11)_N
- net /PEx16_0R(11)_P renamed PEx16_0R(11)_P
- net /PEx16_0R(12)_N renamed PEx16_0R(12)_N
- net /PEx16_0R(12)_P renamed PEx16_0R(12)_P
- net /PEx16_0R(13)_N renamed PEx16_0R(13)_N
- net /PEx16_0R(13)_P renamed PEx16_0R(13)_P
- net /PEx16_0R(14)_N renamed PEx16_0R(14)_N
- net /PEx16_0R(14)_P renamed PEx16_0R(14)_P
- net /PEx16_0R(15)_N renamed PEx16_0R(15)_N
- net /PEx16_0R(15)_P renamed PEx16_0R(15)_P
- net /PEx16_0R(8)_N renamed PEx16_0R(8)_N
- net /PEx16_0R(8)_P renamed PEx16_0R(8)_P
- net /PEx16_0R(9)_N renamed PEx16_0R(9)_N
- net /PEx16_0R(9)_P renamed PEx16_0R(9)_P
- net /PEx16_0T(0)_N renamed PEx16_0T(0)_N
- net /PEx16_0T(0)_P renamed PEx16_0T(0)_P
- net /PEx16_0T(1)_N renamed PEx16_0T(1)_N
- net /PEx16_0T(1)_P renamed PEx16_0T(1)_P
- net /PEx16_0T(2)_N renamed PEx16_0T(2)_N
- net /PEx16_0T(2)_P renamed PEx16_0T(2)_P
- net /PEx16_0T(3)_N renamed PEx16_0T(3)_N
- net /PEx16_0T(3)_P renamed PEx16_0T(3)_P
- net /PEx16_0T(4)_N renamed PEx16_0T(4)_N
- net /PEx16_0T(4)_P renamed PEx16_0T(4)_P
- net /PEx16_0T(5)_N renamed PEx16_0T(5)_N
- net /PEx16_0T(5)_P renamed PEx16_0T(5)_P
- net /PEx16_0T(6)_N renamed PEx16_0T(6)_N
- net /PEx16_0T(6)_P renamed PEx16_0T(6)_P
- net /PEx16_0T(7)_N renamed PEx16_0T(7)_N
- net /PEx16_0T(7)_P renamed PEx16_0T(7)_P
- net /PEx16_CLK_N renamed PEx16_CLK_N
- net /PEx16_CLK_P renamed PEx16_CLK_P
- net /PEx1_0CLK_N renamed PEx1_0CLK_N
- net /PEx1_0CLK_P renamed PEx1_0CLK_P
- net /PEx1_0R_N renamed PEx1_0R_N
- net /PEx1_0R_P renamed PEx1_0R_P
- net /PEx1_0T_N renamed PEx1_0T_N
- net /PEx1_0T_P renamed PEx1_0T_P
- net /PEx1_3CLK_N renamed PEx1_3CLK_N
- net /PEx1_3CLK_P renamed PEx1_3CLK_P
- net /PEx1_3R_N renamed PEx1_3R_N
- net /PEx1_3R_P renamed PEx1_3R_P
- net /PEx1_3T_N renamed PEx1_3T_N
- net /PEx1_3T_P renamed PEx1_3T_P
- net /PEx8_REFCLK1_N renamed PEx8_REFCLK1_N
- net /PEx8_REFCLK1_P renamed PEx8_REFCLK1_P
- net /PEx8_REFCLK2_N renamed PEx8_REFCLK2_N
- net /PEx8_REFCLK2_P renamed PEx8_REFCLK2_P
- net /PSON# renamed /PCIe 104/PSON#
- net /PWRGOOD renamed Net-(J1-Pad46)
- net /SDVO_CLK renamed /PCIe 104/SDVO_CLK
- net /SMB_ALERT renamed SMB_ALERT
- net /SMB_CLK renamed SMB_CLK
- net /SMB_DAT renamed SMB_DAT
- net /STK0 / WAKE# renamed /PCIe 104/STK0 / WAKE#
- net /STK1 / PEG_ENA# renamed /PCIe 104/STK1 / PEG_ENA#
- net /STK2 / SDVO_DAT renamed /PCIe 104/STK2 / SDVO_DAT
- net /USB_0_N renamed /PCIe 104/USB_0_N
- net /USB_0_P renamed /PCIe 104/USB_0_P
- net /USB_1_N renamed /PCIe 104/USB_1_N
- net /USB_1_P renamed /PCIe 104/USB_1_P
- J1 pad 01: /USB_OC -> /PCIe 104/USB_OC
- J1 pad 101: /PEx16_0T(15)_N -> PEx16_0T(15)_N
- J1 pad 11: /PEx1_1T_P -> PEx1_1T_P
- J1 pad 110: /PEx16_0R(0)_P -> PEx16_0R(0)_P
- J1 pad 112: /PEx16_0R(0)_N -> PEx16_0R(0)_N
- J1 pad 116: /PEx16_0R(1)_P -> PEx16_0R(1)_P
- J1 pad 118: /PEx16_0R(1)_N -> PEx16_0R(1)_N
- J1 pad 122: /PEx16_0R(2)_P -> PEx16_0R(2)_P
- J1 pad 124: /PEx16_0R(2)_N -> PEx16_0R(2)_N
- J1 pad 128: /PEx16_0R(3)_P -> PEx16_0R(3)_P
- J1 pad 13: /PEx1_1T_N -> PEx1_1T_N
- J1 pad 130: /PEx16_0R(3)_N -> PEx16_0R(3)_N
- J1 pad 134: /PEx16_0R(4)_P -> PEx16_0R(4)_P
- J1 pad 136: /PEx16_0R(4)_N -> PEx16_0R(4)_N
- J1 pad 140: /PEx16_0R(5)_P -> PEx16_0R(5)_P
- J1 pad 142: /PEx16_0R(5)_N -> PEx16_0R(5)_N
- J1 pad 146: /PEx16_0R(6)_P -> PEx16_0R(6)_P
- J1 pad 148: /PEx16_0R(6)_N -> PEx16_0R(6)_N
- J1 pad 152: /PEx16_0R(7)_P -> PEx16_0R(7)_P
- J1 pad 154: /PEx16_0R(7)_N -> PEx16_0R(7)_N
- J1 pad 17: /PEx1_2T_P -> PEx1_2T_P
- J1 pad 19: /PEx1_2T_N -> PEx1_2T_N
- J1 pad 23: /PEx1_1R_P -> PEx1_1R_P
- J1 pad 25: /PEx1_1R_N -> PEx1_1R_N
- J1 pad 29: /PEx1_2R_P -> PEx1_2R_P
- J1 pad 31: /PEx1_2R_N -> PEx1_2R_N
- J1 pad 35: /PEx1_1CLK_P -> PEx1_1CLK_P
- J1 pad 37: /PEx1_1CLK_N -> PEx1_1CLK_N
- J1 pad 41: /PEx1_2CLK_P -> PEx1_2CLK_P
- J1 pad 43: /PEx1_2CLK_N -> PEx1_2CLK_N
- J1 pad 57: /PEx16_0T(8)_P -> PEx16_0T(8)_P
- J1 pad 59: /PEx16_0T(8)_N -> PEx16_0T(8)_N
- J1 pad 63: /PEx16_0T(9)_P -> PEx16_0T(9)_P
- J1 pad 65: /PEx16_0T(9)_N -> PEx16_0T(9)_N
- J1 pad 69: /PEx16_0T(10)_P -> PEx16_0T(10)_P
- J1 pad 71: /PEx16_0T(10)_N -> PEx16_0T(10)_N
- J1 pad 75: /PEx16_0T(11)_P -> PEx16_0T(11)_P
- J1 pad 77: /PEx16_0T(11)_N -> PEx16_0T(11)_N
- J1 pad 81: /PEx16_0T(12)_P -> PEx16_0T(12)_P
- J1 pad 83: /PEx16_0T(12)_N -> PEx16_0T(12)_N
- J1 pad 87: /PEx16_0T(13)_P -> PEx16_0T(13)_P
- J1 pad 89: /PEx16_0T(13)_N -> PEx16_0T(13)_N
- J1 pad 93: /PEx16_0T(14)_P -> PEx16_0T(14)_P
- J1 pad 95: /PEx16_0T(14)_N -> PEx16_0T(14)_N
- J1 pad 99: /PEx16_0T(15)_P -> PEx16_0T(15)_P
- J10 pad SH1: unconnected-(J10-SHIELD-PadSH1) -> GND
- J10 pad SH2: unconnected-(J10-SHIELD__1-PadSH2) -> GND
- J2 pad A16: /PEx16_0R(0)_P -> PEx16_0R(0)_P
- J2 pad A17: /PEx16_0R(0)_N -> PEx16_0R(0)_N
- J2 pad A21: /PEx16_0R(1)_P -> PEx16_0R(1)_P
- J2 pad A22: /PEx16_0R(1)_N -> PEx16_0R(1)_N
- J2 pad A25: /PEx16_0R(2)_P -> PEx16_0R(2)_P
- J2 pad A26: /PEx16_0R(2)_N -> PEx16_0R(2)_N
- J2 pad A29: /PEx16_0R(3)_P -> PEx16_0R(3)_P
- J2 pad A30: /PEx16_0R(3)_N -> PEx16_0R(3)_N
- J2 pad A35: /PEx16_0R(4)_P -> PEx16_0R(4)_P
- J2 pad A36: /PEx16_0R(4)_N -> PEx16_0R(4)_N
- J2 pad A39: /PEx16_0R(5)_P -> PEx16_0R(5)_P
- J2 pad A40: /PEx16_0R(5)_N -> PEx16_0R(5)_N
- J2 pad A43: /PEx16_0R(6)_P -> PEx16_0R(6)_P
- J2 pad A44: /PEx16_0R(6)_N -> PEx16_0R(6)_N
- J2 pad A47: /PEx16_0R(7)_P -> PEx16_0R(7)_P
- J2 pad A48: /PEx16_0R(7)_N -> PEx16_0R(7)_N
- J2 pad B10: +3.3VA -> +3.3V
- J6 pad B10: +3.3VA -> +3.3V
- J6 pad B14: /PEx16_0R(0)_P -> PEx16_0T(8)_P
- J6 pad B15: /PEx16_0R(0)_N -> PEx16_0T(8)_N
- J6 pad B19: /PEx16_0R(1)_P -> PEx16_0T(9)_P
- J6 pad B20: /PEx16_0R(1)_N -> PEx16_0T(9)_N
- J6 pad B23: /PEx16_0R(2)_P -> PEx16_0T(10)_P
- J6 pad B24: /PEx16_0R(2)_N -> PEx16_0T(10)_N
- J6 pad B27: /PEx16_0R(3)_P -> PEx16_0T(11)_P
- J6 pad B28: /PEx16_0R(3)_N -> PEx16_0T(11)_N
- J6 pad B33: /PEx16_0R(4)_P -> PEx16_0T(12)_P
- J6 pad B34: /PEx16_0R(4)_N -> PEx16_0T(12)_N
- J6 pad B37: /PEx16_0R(5)_P -> PEx16_0T(13)_P
- J6 pad B38: /PEx16_0R(5)_N -> PEx16_0T(13)_N
- J6 pad B41: /PEx16_0R(6)_P -> PEx16_0T(14)_P
- J6 pad B42: /PEx16_0R(6)_N -> PEx16_0T(14)_N
- J6 pad B45: /PEx16_0R(7)_P -> PEx16_0T(15)_P
- J6 pad B46: /PEx16_0R(7)_N -> PEx16_0T(15)_N
- J7 pad 75: GND -> unconnected-(J7-P75-Pad75)
- J7 pad SH1: unconnected-(J7-SHIELD-PadSH1) -> GND
- J7 pad SH2: unconnected-(J7-SHIELD__1-PadSH2) -> GND
- J8 pad 41: /PEx1_2R_N -> PEx1_1R_P
- J8 pad 43: /PEx1_2R_P -> PEx1_1R_N
- J8 pad 47: /PEx1_2T_N -> PEx1_1T_P
- J8 pad 49: /PEx1_2T_P -> PEx1_1T_N
- J8 pad 53: /PEx1_2CLK_N -> PEx1_1CLK_N
- J8 pad 55: /PEx1_2CLK_P -> PEx1_1CLK_P
- J8 pad SH1: unconnected-(J8-SHIELD-PadSH1) -> GND
- J8 pad SH2: unconnected-(J8-SHIELD__1-PadSH2) -> GND
- J9 pad 41: /PEx1_1R_N -> PEx1_2R_P
- J9 pad 43: /PEx1_1R_P -> PEx1_2R_N
- J9 pad 47: /PEx1_1T_N -> PEx1_2T_P
- J9 pad 49: /PEx1_1T_P -> PEx1_2T_N
- J9 pad 53: /PEx1_1CLK_N -> PEx1_2CLK_N
- J9 pad 55: /PEx1_1CLK_P -> PEx1_2CLK_P
- J9 pad SH1: unconnected-(J9-SHIELD-PadSH1) -> GND
- J9 pad SH2: unconnected-(J9-SHIELD__1-PadSH2) -> GND
Routing:
- net PEx16_0T(7)_N: track 0.00 -> 123.5 mm, vias 0 -> 2
- net PEx16_0T(7)_P: track 0.00 -> 123.4 mm, vias 0 -> 2
- net PEx16_0T(6)_P: track 0.00 -> 123.2 mm, vias 0 -> 2
- net PEx16_0T(6)_N: track 0.00 -> 123.2 mm, vias 0 -> 2
- net PEx16_0T(5)_N: track 0.00 -> 123.1 mm, vias 0 -> 2
- net PEx16_0T(5)_P: track 0.00 -> 123.1 mm, vias 0 -> 2
- net PEx16_0T(4)_P: track 0.00 -> 122.5 mm, vias 0 -> 2
- net PEx16_0T(4)_N: track 0.00 -> 122.5 mm, vias 0 -> 2
- net PEx16_0T(3)_P: track 0.00 -> 121.0 mm, vias 0 -> 2
- net PEx16_0T(3)_N: track 0.00 -> 121.0 mm, vias 0 -> 2
- net PEx16_0T(1)_N: track 0.00 -> 120.1 mm, vias 0 -> 2
- net PEx16_0T(2)_N: track 0.00 -> 120.0 mm, vias 0 -> 2
- net PEx16_0T(1)_P: track 0.00 -> 120.0 mm, vias 0 -> 2
- net PEx16_0T(2)_P: track 0.00 -> 119.9 mm, vias 0 -> 2
- net PEx16_0T(0)_N: track 0.00 -> 119.4 mm, vias 0 -> 2
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- added copper zone on In1.Cu, net GND
- added copper zone on F.Cu, net Net-(U2-SW)
Other:
- copper layers 2 -> 4
