File: PCI_104_PCIE_Adapterboard.kicad_pcb (KiCad board)
At the start: 4 copper layers, 70 parts, among them J1 ASP-129637-03, J10 1-2199119-5, J11 Conn_01x02_Pin, J2 10061913-102PLF, J3 Conn_01x02_Pin, J4 Conn_01x02_Pin, J5 Conn_01x02_Pin, J6 10061913-102PLF, J7 1-2199119-5, J8 1-2199119-5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

Commit message: layout done!!
Parts:
- added C33: 100uF, Capacitor_SMD:C_1206_3216Metric, F.Cu at (121.9, 143.1)
- added C34: 100uF, Capacitor_SMD:C_1206_3216Metric, F.Cu at (112.0, 143.2)
- added C35: 100uF, Capacitor_SMD:C_1206_3216Metric, F.Cu at (121.9, 139.7)
- added C36: 100uF, Capacitor_SMD:C_1206_3216Metric, F.Cu at (112.0, 139.7)
- added C37: 100uF, Capacitor_SMD:C_1206_3216Metric, F.Cu at (122.1, 131.5)
- added C38: 100uF, Capacitor_SMD:C_1206_3216Metric, F.Cu at (122.1, 135.1)
- added C39: 100uF, Capacitor_SMD:C_1206_3216Metric, F.Cu at (112.0, 131.5)
- added C40: 100uF, Capacitor_SMD:C_1206_3216Metric, F.Cu at (112.0, 135.6)
- added H5: MountingHole_Pad, MountingHole:MountingHole_3.2mm_M3_Pad_TopBottom, F.Cu at (12.0, 139.4)
- added H6: MountingHole_Pad, MountingHole:MountingHole_3.2mm_M3_Pad_TopBottom, F.Cu at (12.0, 164.4)
- added H7: MountingHole_Pad, MountingHole:MountingHole_3.2mm_M3_Pad_TopBottom, F.Cu at (221.9, 164.4)
- added H8: MountingHole_Pad, MountingHole:MountingHole_3.2mm_M3_Pad_TopBottom, F.Cu at (221.9, 139.4)
- added J12: Conn_02x02_Top_Bottom, Connector_Molex:Molex_Mini-Fit_Jr_5569-04A1_2x02_P4.20mm_Horizontal, F.Cu at (122.6, 188.5)
- C12, C13, C16, C2, C3, C4, C5, C7, C8: footprint Capacitor_SMD:C_0603_1608Metric -> Capacitor_SMD:C_0402_1005Metric
- C14: footprint Capacitor_SMD:C_0805_2012Metric_Pad1.18x1.45mm_HandSolder -> Capacitor_SMD:C_0402_1005Metric
- C15: footprint Capacitor_SMD:C_0603_1608Metric -> Resistor_SMD:R_0402_1005Metric
- C17, C18, C19, C20: value 47uF -> 100uF; footprint Capacitor_SMD:C_0805_2012Metric_Pad1.18x1.45mm_HandSolder -> Capacitor_SMD:C_1206_3216Metric
- L1: value 150nH -> 260nH; footprint footprints:INDPM5350X200N -> Inductor_SMD:L_Coilcraft_XAL1010-XXX
- R10, R12, R15, R16, R17, R3, R4, R5, R6, R7, R8, R9: footprint Resistor_SMD:R_0603_1608Metric_Pad0.98x0.95mm_HandSolder -> Resistor_SMD:R_0402_1005Metric
- R11: value 243k -> 205k; footprint Resistor_SMD:R_0603_1608Metric_Pad0.98x0.95mm_HandSolder -> Resistor_SMD:R_0402_1005Metric
- R13: value 100k -> 10k; footprint Resistor_SMD:R_0603_1608Metric_Pad0.98x0.95mm_HandSolder -> Resistor_SMD:R_0402_1005Metric
- R14: value 7.32k -> 8.06k; footprint Resistor_SMD:R_0603_1608Metric_Pad0.98x0.95mm_HandSolder -> Resistor_SMD:R_0402_1005Metric
- moved C21 245.4 mm to (84.2, 171.7), turned to 90 degrees
- moved C22 242.1 mm to (86.2, 171.7), turned to 90 degrees
- moved J4 227.1 mm to (91.2, 22.2), turned to 90 degrees
- moved J5 225.2 mm to (82.5, 22.2), turned to 90 degrees
- moved C27 224.9 mm to (83.3, 146.9), turned to 90 degrees
- moved J3 224.9 mm to (73.7, 22.2), turned to 90 degrees
- moved TP1 224.8 mm to (100.2, 22.0), turned to 90 degrees
- moved TP3 223.0 mm to (104.8, 22.0), turned to 90 degrees
- moved C28 221.9 mm to (85.2, 146.9), turned to 90 degrees
- moved TP2 217.4 mm to (109.4, 22.0), turned to 90 degrees
- moved C12 217.0 mm to (112.6, 166.2), turned to 90 degrees
- moved C13 215.9 mm to (113.6, 166.2), turned to 90 degrees
- moved C7 207.1 mm to (119.2, 166.2), turned to 90 degrees
- moved C8 206.1 mm to (120.1, 166.2), turned to 90 degrees
- moved C18 204.8 mm to (112.0, 146.6), turned to 180 degrees
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Connections:
- J1 pad 03: +3.3VA -> unconnected-(J1-Pad03)
- J1 pad 04: +3.3VA -> unconnected-(J1-Pad04)
- J1 pad 39: +5VA -> unconnected-(J1-Pad39)
- J1 pad 40: +5VA -> unconnected-(J1-Pad40)
- J1 pad G1: +5V -> unconnected-(J1A-GND1-PadG1)
- J1 pad G2: +5V -> unconnected-(J1B-GND2-PadG2)
- J2 pad B4: Net-(J2-PadB4) -> GND
- J2 pad B7: Net-(J2-PadB4) -> GND
- J6 pad B4: Net-(J6-PadB4) -> GND
- J6 pad B7: Net-(J6-PadB4) -> GND
Routing:
- net GND: track 0.00 -> 523.8 mm, vias 0 -> 295
- net SMB_CLK: track 0.00 -> 328.1 mm, vias 0 -> 8
- net SMB_DAT: track 0.00 -> 321.7 mm, vias 0 -> 9
- net SMB_ALERT: track 0.00 -> 228.8 mm, vias 0 -> 4
- net PE_RST#: track 0.00 -> 126.5 mm, vias 0 -> 3
- net /PCIe 104/USB_OC: track 0.00 -> 109.7 mm, vias 0 -> 1
- net /PCIe 104/PSON#: track 0.00 -> 83.0 mm, vias 0 -> 1
- net /PCIe 104/STK0 / WAKE#: track 0.00 -> 82.4 mm, vias 0 -> 1
- net +12V: track 0.00 -> 78.9 mm, vias 0 -> 15
- net /PCIe 104/STK1 / PEG_ENA#: track 0.00 -> 73.8 mm, vias 0 -> 1
- net Net-(J1-Pad46): track 0.00 -> 73.6 mm
- net PEx8_REFCLK1_N: track 0.00 -> 73.5 mm, vias 0 -> 2
- net PEx8_REFCLK1_P: track 0.00 -> 73.3 mm, vias 0 -> 2
- net +3.3V: track 0.00 -> 70.8 mm, vias 0 -> 69
- net PEx16_CLK_N: track 0.00 -> 52.0 mm, vias 0 -> 2
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- added copper zone on F.Cu, net +12V
- added copper zone on In2.Cu, net +12V
- added copper zone on F.Cu, net +3.3V
- added copper zone on In2.Cu, net +3.3V
- added copper zone on B.Cu, net +5V
- added copper zone on F.Cu, net +5V
- added copper zone on F.Cu, net GND
- added copper zone on In4.Cu, net GND
Other:
- board outline added: 240 x 192.9 mm
- copper layers 4 -> 6

Commit message: layout complete
Parts:
- added C41: 0.01uF, Capacitor_SMD:C_0402_1005Metric, F.Cu at (164.4, 140.2)
- added C42: 0.01uF, Capacitor_SMD:C_0402_1005Metric, F.Cu at (152.2, 137.1)
- added C43: 0.01uF, Capacitor_SMD:C_0402_1005Metric, F.Cu at (151.4, 140.1)
- C15: footprint Resistor_SMD:R_0402_1005Metric -> Capacitor_SMD:C_0402_1005Metric
- moved C24 82.4 mm to (190.0, 226.6)
- moved C26 82.4 mm to (190.1, 201.6)
- moved J8 82.4 mm to (182.2, 236.3)
- moved C23 82.4 mm to (188.1, 226.6)
- moved C25 82.4 mm to (188.1, 201.6)
- moved H7 82.4 mm to (262.2, 236.3)
- moved J9 82.4 mm to (182.2, 211.2)
- moved H8 82.4 mm to (262.2, 211.2)
- moved C17 65.6 mm to (152.3, 201.8)
- moved C18 65.6 mm to (152.3, 198.4)
- moved C3 65.6 mm to (197.6, 159.1)
- moved C31 65.6 mm to (262.6, 146.1)
- moved C34 65.6 mm to (152.3, 194.9)
- moved C36 65.6 mm to (152.3, 191.5)
- moved H2 65.6 mm to (161.0, 85.0)
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Routing:
- net /PCIe 104/PSON#: track 83.0 -> 109.4 mm
- net Net-(C43-Pad1): track 73.6 -> 99.9 mm
- net /PCIe 104/USB_OC: track 109.7 -> 134.5 mm
- net /PCIe 104/STK1 / PEG_ENA#: track 73.8 -> 98.6 mm
- net /PCIe 104/STK0 / WAKE#: track 82.4 -> 107.1 mm
- net /PCIe 104/SDVO_CLK: track 42.8 -> 66.8 mm
- net /PCIe 104/STK2 / SDVO_DAT: track 44.0 -> 67.5 mm
- net PEx1_1CLK_P: track 80.8 -> 102.8 mm
- net PEx1_2CLK_P: track 61.7 -> 83.3 mm
- net PEx1_2T_P: track 49.2 -> 69.9 mm
- net PEx1_2T_N: track 49.2 -> 69.9 mm
- net PEx1_1R_P: track 78.3 -> 99.0 mm
- net PEx1_1T_N: track 71.1 -> 91.8 mm
- net PEx1_1T_P: track 71.1 -> 91.8 mm
- net PEx1_1CLK_N: track 82.2 -> 102.9 mm
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Other:
- board size 240 x 192.9 mm -> 240 x 233.2 mm
- board text added: "CLK"
- board text added: "DAT"
- board text added: "PCIe/104 to PCIe Adapter"
- board text added: "PEG_ENA#"
- board text added: "PSON#"
- board text added: "PWRGOOD"
- board text added: "SDVO"
- board text added: "USB_OC"
- board text added: "WAKE#"
- board text added: "With Bifurcation"

Commit message: stitched gnd planes
Routing:
- net GND: vias 298 -> 463
