File: PCI_104_PCIE_Adapterboard.kicad_sch (KiCad schematic)
At the start: 53 parts, among them J1 ASP-129637-03, J10 1-2199119-5, J2 10061913-102PLF, J3 Conn_01x02_Pin, J4 Conn_01x02_Pin, J5 Conn_01x02_Pin, J6 10061913-102PLF, J7 1-2199119-5, J8 1-2199119-5, J9 1-2199119-5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

Commit message: finished schem
Parts:
- removed C1: 10uF, Capacitor_SMD:C_0805_2012Metric_Pad1.18x1.45mm_HandSolder, symbol Device:C_Small
- removed C10, C11, C6, C9: 10uF, Capacitor_SMD:C_0805_2012Metric_Pad1.18x1.45mm_HandSolder, symbol Device:C
- removed C12, C7: 1uF, Capacitor_SMD:C_0201_0603Metric_Pad0.64x0.40mm_HandSolder, symbol Device:C
- removed C13, C16, C8: 100nF, Capacitor_SMD:C_0201_0603Metric_Pad0.64x0.40mm_HandSolder, symbol Device:C
- removed C14: 2.2uF, Capacitor_SMD:C_0805_2012Metric_Pad1.18x1.45mm_HandSolder, symbol Device:C
- removed C15: 68nF, Capacitor_SMD:C_0201_0603Metric_Pad0.64x0.40mm_HandSolder, symbol Device:C
- removed C17, C18, C19, C20: 47uF, Capacitor_SMD:C_0805_2012Metric_Pad1.18x1.45mm_HandSolder, symbol Device:C
- removed C2: 1uF, Capacitor_SMD:C_0201_0603Metric_Pad0.64x0.40mm_HandSolder, symbol Device:C_Small
- removed C3, C4, C5: 0.1uF, Capacitor_SMD:C_0201_0603Metric_Pad0.64x0.40mm_HandSolder, symbol Device:C_Small
- removed J1: ASP-129637-03, footprints:SAMTEC_ASP-129637-03, symbol ASP-129637-03:ASP-129637-03
- removed J10, J7, J8, J9: 1-2199119-5, footprints:TE_1-2199119-5, symbol 1-2199119-5:1-2199119-5
- removed J2, J6: 10061913-102PLF, footprints:AMPHENOL_10061913-102PLF, symbol 10061913-102PLF:10061913-102PLF
- removed J3, J4, J5: Conn_01x02_Pin, Connector_PinHeader_2.54mm:PinHeader_1x02_P2.54mm_Vertical, symbol Connector:Conn_01x02_Pin
- removed L1: 150nH, symbol Device:L
- removed R1, R2: R_US, Resistor_SMD:R_0603_1608Metric_Pad0.98x0.95mm_HandSolder, symbol Device:R_US
- removed R10, R7, R8, R9: 50, Resistor_SMD:R_0603_1608Metric_Pad0.98x0.95mm_HandSolder, symbol Device:R_Small_US
- removed R11: 243k, Resistor_SMD:R_0603_1608Metric_Pad0.98x0.95mm_HandSolder, symbol Device:R_US
- removed R12, R13: 100k, Resistor_SMD:R_0603_1608Metric_Pad0.98x0.95mm_HandSolder, symbol Device:R_US
- removed R14: 7.32k, Resistor_SMD:R_0603_1608Metric_Pad0.98x0.95mm_HandSolder, symbol Device:R_US
- removed R15: 4.99k, Resistor_SMD:R_0603_1608Metric_Pad0.98x0.95mm_HandSolder, symbol Device:R_US
- removed R16: 56.2k, Resistor_SMD:R_0603_1608Metric_Pad0.98x0.95mm_HandSolder, symbol Device:R_US
- removed R17: 10k, Resistor_SMD:R_0603_1608Metric_Pad0.98x0.95mm_HandSolder, symbol Device:R_US
- removed R3, R4, R5, R6: 33, Resistor_SMD:R_0603_1608Metric_Pad0.98x0.95mm_HandSolder, symbol Device:R_Small_US
- removed TP1: PWRGOOD, TestPoint:TestPoint_Keystone_5015_Micro_Mini, symbol Connector:TestPoint
- removed TP2, TP3: TestPoint, TestPoint:TestPoint_Keystone_5015_Micro_Mini, symbol Connector:TestPoint
- removed U1: ZL40264LDG1, QFN_264LDG1_MCH, symbol ZL40264:ZL40264LDG1
- removed U2: TPS54KB21RZRR, RZR0016A-MFG, symbol TPS54KB21RZRR:TPS54KB21RZRR
Connections:
- no-connect marks 174 -> 0
Other:
- added sheet Bifurcation (bifurcation.kicad_sch)
- added sheet M.2 NVME (m2_nvme.kicad_sch)
- added sheet PCIe 104 (pcie_104.kicad_sch)
- added sheet Power (power.kicad_sch)
- note removed: "Add capacitors"
- note removed: "Any Device that uses the x16 Link attaches PEG_ENA to ground"
- company: (none) -> By Madhav Kapa
- title: (none) -> PCIe/104 Adapter

Commit message: layout done!!
Other:
- note added: "Stackup: JLC06161H-3313"
Changed lines of the file:
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@@
 		(company "By Madhav Kapa")
+	)
+	(text "Stackup: JLC06161H-3313"
+		(exclude_from_sim no)
+		(at 40.132 65.786 0)
+		(effects
+			(font
+				(size 2.54 2.54)
+			)
+		)
 	)
 	(sheet
