File: m2_nvme.kicad_sch (KiCad schematic)
At the start: 12 parts, among them J10 1-2199119-5, J7 1-2199119-5, J8 1-2199119-5, J9 1-2199119-5

Commit message: pcie traces routed
Parts:
- renumbered J9 to J8, J8 to J9
Connections:
- net GND: now also J10.SH1 (SHIELD), J10.SH2 (SHIELD__1), J7.SH1 (SHIELD), J7.SH2 (SHIELD__1), J8.SH1 (SHIELD), J8.SH2 (SHIELD__1), J9.SH1 (SHIELD), J9.SH2 (SHIELD__1)
- net PEx1_1R_N: now also J8.43 (P43); no longer J8.41 (P41)
- net PEx1_1R_P: now also J8.41 (P41); no longer J8.43 (P43)
- net PEx1_1T_N: now also J8.49 (P49); no longer J8.47 (P47)
- net PEx1_1T_P: now also J8.47 (P47); no longer J8.49 (P49)
- net PEx1_2R_N: now also J9.43 (P43); no longer J9.41 (P41)
- net PEx1_2R_P: now also J9.41 (P41); no longer J9.43 (P43)
- net PEx1_2T_N: now also J9.49 (P49); no longer J9.47 (P47)
- net PEx1_2T_P: now also J9.47 (P47); no longer J9.49 (P49)

Commit message: layout done!!
Parts:
- added H5, H6, H7, H8: MountingHole_Pad, MountingHole:MountingHole_3.2mm_M3_Pad_TopBottom, symbol Mechanical:MountingHole_Pad
Connections:
- no-connect marks 140 -> 145
