File: pcie_104.kicad_sch (KiCad schematic)
At the start: 9 parts, among them J1 ASP-129637-03, J3 Conn_01x02_Pin, J4 Conn_01x02_Pin, J5 Conn_01x02_Pin

Commit message: pcie traces routed
Parts:
- added J11: Conn_01x02_Pin, Connector_PinHeader_2.54mm:PinHeader_1x02_P2.54mm_Vertical, symbol Connector:Conn_01x02_Pin
Connections:
- net GND: now also J11.2 (Pin_2)
- net USB_OC: now also J11.1 (Pin_1)
Other:
- moved on the sheet: J1A, J1B, J1C, J3, J4, J5, R1, R2, TP1, TP2, TP3

Commit message: layout done!!
Parts:
- added H1, H2, H3, H4: MountingHole_Pad, MountingHole:MountingHole_3.2mm_M3_Pad_TopBottom, symbol Mechanical:MountingHole_Pad
Connections:
- net GND: now also H1.1, H2.1, H3.1, H4.1
- net +3.3VA: no longer names the net of J1.03
- net +3.3VA: no longer J1.04
- net +5V: no longer names the net of J1.G1 (GND1)
- net +5V: no longer J1.G2 (GND2)
- net +5VA: no longer names the net of J1.39
- net +5VA: no longer J1.40
- no-connect marks 0 -> 6
Other:
- note added: "3.3V provided not used"
- note added: "5V always on not needed"

Commit message: layout complete
Parts:
- added C41, C42, C43: 0.01uF, Capacitor_SMD:C_0402_1005Metric, symbol Device:C
Connections:
- net DIR: now also C41.1
- net GND: now also C41.2, C42.2, C43.2
- net PSON#: now also C42.1
- net at J1.46, TP1.1: now also C43.1
Other:
- moved on the sheet: J1B, J1C, J3, J4, J5, R1, R2, TP1, TP2, TP3
