File: power.kicad_sch (KiCad schematic)
At the start: 24 parts, among them U2 TPS54KB21RZRR

Commit message: pcie traces routed
Parts:
- C15, C16: footprint Capacitor_SMD:C_0201_0603Metric_Pad0.64x0.40mm_HandSolder -> Capacitor_SMD:C_0603_1608Metric
- L1: footprint (none) -> footprints:INDPM5350X200N
Changed lines of the file:
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@@
 			)
 		)
-		(property "Footprint" ""
+		(property "Footprint" "footprints:INDPM5350X200N"
 			(at 207.01 44.45 0)
 			(effects
@@
 			)
 		)
-		(property "Footprint" "Capacitor_SMD:C_0201_0603Metric_Pad0.64x0.40mm_HandSolder"
+		(property "Footprint" "Capacitor_SMD:C_0603_1608Metric"
 			(at 135.5852 83.82 0)
 			(effects
@@
 			)
 		)
-		(property "Footprint" "Capacitor_SMD:C_0201_0603Metric_Pad0.64x0.40mm_HandSolder"
+		(property "Footprint" "Capacitor_SMD:C_0603_1608Metric"
 			(at 203.2 35.8648 0)
 			(effects

Commit message: layout done!!
Parts:
- added C33, C34, C35, C36, C37, C38, C39, C40: 100uF, Capacitor_SMD:C_1206_3216Metric, symbol Device:C
- added J12: Conn_02x02_Top_Bottom, Connector_Molex:Molex_Mini-Fit_Jr_5569-04A1_2x02_P4.20mm_Horizontal, symbol Connector_Generic:Conn_02x02_Top_Bottom
- C12, C13, C16, C7, C8: footprint Capacitor_SMD:C_0603_1608Metric -> Capacitor_SMD:C_0402_1005Metric
- C14: footprint Capacitor_SMD:C_0805_2012Metric_Pad1.18x1.45mm_HandSolder -> Capacitor_SMD:C_0402_1005Metric
- C15: footprint Capacitor_SMD:C_0603_1608Metric -> Resistor_SMD:R_0402_1005Metric
- C17, C18, C19, C20: value 47uF -> 100uF; footprint Capacitor_SMD:C_0805_2012Metric_Pad1.18x1.45mm_HandSolder -> Capacitor_SMD:C_1206_3216Metric
- L1: value 150nH -> 260nH; footprint footprints:INDPM5350X200N -> Inductor_SMD:L_Coilcraft_XAL1010-XXX
- R11: value 243k -> 205k; footprint Resistor_SMD:R_0603_1608Metric_Pad0.98x0.95mm_HandSolder -> Resistor_SMD:R_0402_1005Metric
- R12, R15, R16, R17: footprint Resistor_SMD:R_0603_1608Metric_Pad0.98x0.95mm_HandSolder -> Resistor_SMD:R_0402_1005Metric
- R13: value 100k -> 10k; footprint Resistor_SMD:R_0603_1608Metric_Pad0.98x0.95mm_HandSolder -> Resistor_SMD:R_0402_1005Metric
- R14: value 7.32k -> 8.06k; footprint Resistor_SMD:R_0603_1608Metric_Pad0.98x0.95mm_HandSolder -> Resistor_SMD:R_0402_1005Metric
Connections:
- net +3.3V: now also C33.1, C34.1, C35.1, C36.1, C37.1, C38.1, C39.1, C40.1
- net +5V: now also J12.3 (Pin_3), J12.4 (Pin_4)
- net GND: now also C33.2, C34.2, C35.2, C36.2, C37.2, C38.2, C39.2, C40.2, J12.1 (Pin_1), J12.2 (Pin_2)

Commit message: layout complete
Parts:
- C15: footprint Resistor_SMD:R_0402_1005Metric -> Capacitor_SMD:C_0402_1005Metric
Changed lines of the file:
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@@
 			)
 		)
-		(property "Footprint" "Resistor_SMD:R_0402_1005Metric"
+		(property "Footprint" "Capacitor_SMD:C_0402_1005Metric"
 			(at 135.5852 83.82 0)
 			(effects
